Commit message: Added custom coffee top

File: src/start_creating_robots/worlds_and_models/krytn/krytn.urdf.xacro (robot description, xacro)
@@ -1,8 +1,8 @@
 <?xml version='1.0' encoding='utf-8'?>
-<robot xmlns:xacro="http://www.ros.org/wiki/xacro" name="krytn" >
+<robot xmlns:xacro="http://www.ros.org/wiki/xacro" name="krytn">
     <xacro:arg name="with_sensors" default="true" />
     <!-- Include the robot base. Configure it with a differential drive control plugin -->
     <xacro:include filename="$(find start_creating_robots)/worlds_and_models/krytn/magni.urdf.xacro" />
-    <xacro:if value="$(arg with_sensors)" >
+    <xacro:if value="$(arg with_sensors)">
         <!-- Include an extra 2D Lidar -->
         <xacro:include filename="$(find start_creating_robots)/worlds_and_models/krytn/lidar_2d_v1.urdf.xacro" />
@@ -10,37 +10,44 @@
         <xacro:include filename="$(find start_creating_robots)/worlds_and_models/krytn/realsense_d435.urdf.xacro" />
     </xacro:if>
+    <!-- Coffee Holder Top -->
+    <link name="krytn_top">
+        <visual name="visual">
+            <geometry>
+                <mesh filename="file://$(find start_creating_robots)/worlds_and_models/krytn/meshes/krytn_v2-Body.dae"/>
+            </geometry>
+        </visual>
+    </link>
+    <joint class="krytn_top_joint" type="fixed">
+        <parent link="base_footprint"/>
+        <child link="krytn_top"/>
+        <origin xyz="0.05 0 0.26" rpy="0 0 1.57"/>
+    </joint>
     <!-- Gazebo specific plugins-->
     <gazebo >
-        <xacro:if value="$(arg with_sensors)" >
-            <plugin
-            filename="ignition-gazebo-sensors-system"
-            name="ignition::gazebo::systems::Sensors">
+        <xacro:if value="$(arg with_sensors)">
+            <plugin filename="ignition-gazebo-sensors-system" name="ignition::gazebo::systems::Sensors">
                 <render_engine>ogre2</render_engine>
             </plugin>
         </xacro:if>
         <!-- Publish joints for robot description tf publisher. -->
-        <plugin
-            filename="ignition-gazebo-joint-state-publisher-system"
-            name="ignition::gazebo::systems::JointStatePublisher">
+        <plugin filename="ignition-gazebo-joint-state-publisher-system" name="ignition::gazebo::systems::JointStatePublisher">
             <topic>joint_states</topic>
         </plugin>
         <!-- Plugin to allow Gazebo to recieve cmd_vel and rotate wheels in Gazebo. -->
-        <plugin
-                filename="ignition-gazebo-diff-drive-system"
-                name="ignition::gazebo::systems::DiffDrive">
-                <left_joint>left_wheel_joint</left_joint>
-                <right_joint>right_wheel_joint</right_joint>
-                <frame_id>odom</frame_id>
-                <wheel_separation>0.326</wheel_separation>
-                <wheel_radius>0.128</wheel_radius>
-                <odom_publish_frequency>20</odom_publish_frequency>
-                <max_linear_acceleration>1</max_linear_acceleration>
-                <min_linear_acceleration>-1</min_linear_acceleration>
-                <max_angular_acceleration>2</max_angular_acceleration>
-                <min_angular_acceleration>-2</min_angular_acceleration>
-                <max_linear_velocity>0.5</max_linear_velocity>
-                <min_linear_velocity>-0.5</min_linear_velocity>
-                <max_angular_velocity>1</max_angular_velocity>
-                <min_angular_velocity>-1</min_angular_velocity>
+        <plugin filename="ignition-gazebo-diff-drive-system" name="ignition::gazebo::systems::DiffDrive">
+            <left_joint>left_wheel_joint</left_joint>
+            <right_joint>right_wheel_joint</right_joint>
+            <frame_id>odom</frame_id>
+            <wheel_separation>0.326</wheel_separation>
+            <wheel_radius>0.128</wheel_radius>
+            <odom_publish_frequency>20</odom_publish_frequency>
+            <max_linear_acceleration>1</max_linear_acceleration>
+            <min_linear_acceleration>-1</min_linear_acceleration>
+            <max_angular_acceleration>2</max_angular_acceleration>
+            <min_angular_acceleration>-2</min_angular_acceleration>
+            <max_linear_velocity>0.5</max_linear_velocity>
+            <min_linear_velocity>-0.5</min_linear_velocity>
+            <max_angular_velocity>1</max_angular_velocity>
+            <min_angular_velocity>-1</min_angular_velocity>
         </plugin>
     </gazebo>

Commit message: xml checked

File: src/start_creating_robots/worlds_and_models/krytn/krytn.urdf.xacro (robot description, xacro)
@@ -14,12 +14,12 @@
         <visual name="visual">
             <geometry>
-                <mesh filename="file://$(find start_creating_robots)/worlds_and_models/krytn/meshes/krytn_v2-Body.dae"/>
+                <mesh filename="file://$(find start_creating_robots)/worlds_and_models/krytn/meshes/krytn_coffee_top.dae"/>
             </geometry>
         </visual>
     </link>
     <joint class="krytn_top_joint" type="fixed">
-        <parent link="base_footprint"/>
-        <child link="krytn_top"/>
-        <origin xyz="0.05 0 0.26" rpy="0 0 1.57"/>
+        <parent link="base_footprint" />
+        <child link="krytn_top" />
+        <origin xyz="0.05 0 0.26" rpy="0 0 1.57" />
     </joint>
     <!-- Gazebo specific plugins-->

Commit message: added coffee holder

File: src/start_creating_robots/worlds_and_models/krytn/krytn.urdf.xacro (robot description, xacro)
@@ -18,5 +18,5 @@
         </visual>
     </link>
-    <joint class="krytn_top_joint" type="fixed">
+    <joint name="krytn_top_joint" type="fixed">
         <parent link="base_footprint" />
         <child link="krytn_top" />
